File: piano-monitor.kicad_pcb (KiCad board)
At the start: 2 copper layers, 166 x 72.3 mm, 7 parts, among them J3 NCJ6FA-V, J4 DC, J7 NCJ6FA-V

Commit message: Finalise the AMP pcb
Parts:
- added J2: Conn_01x03, Connector_PinHeader_2.54mm:PinHeader_1x03_P2.54mm_Vertical, F.Cu at (115.2, 86.2)
- added LS1: Speaker, Connector_PinHeader_2.54mm:PinHeader_1x02_P2.54mm_Vertical, F.Cu at (147.7, 58.0)
- added LS2: Speaker, Connector_PinHeader_2.54mm:PinHeader_1x02_P2.54mm_Vertical, F.Cu at (127.5, 58.0)
- moved J4 11.3 mm to (164.0, 84.5)
Connections:
- net T1 renamed Right
- net T2 renamed Left
- J4 pad 1: GND -> S1
Routing:
- net S1: track 84.3 -> 0.00 mm
- net Right: track 37.1 -> 58.4 mm
- net Left: track 35.5 -> 49.8 mm
- net Net-(LS2-Pad1): track 0.00 -> 3.30 mm
- net Net-(U1-R-): track 0.00 -> 3.24 mm
- net Net-(LS1-Pad1): track 0.00 -> 3.17 mm
- net Net-(U1-L-): track 0.00 -> 3.10 mm
- net +24V: track 16.9 -> 15.4 mm
- added copper zone on B.Cu, net S1
- removed copper zone on B.Cu, net GND
Other:
- outline, holes or cut-outs redrawn
- board text added: "#287"
- board text added: "FEB 26"
- board text added: "L+"
- board text added: "R+"
